File: Hardware/Joystick_Follower_Hat/Joystick_Follower_Hat.sch (KiCad schematic (older format))
At the start: 21 parts, among them SW1 SW_Push, SW2 SW_Push, SW3 SW_Push, SW4 SW_Push, U1 COM-09032

Commit message: PCB Files and Gerber Files
Parts:
- U1: symbol COM-09032:COM-09032 -> Joystick_Follower_Hat-rescue:COM-09032-COM-09032
Changed lines of the file:
@@
 $EndComp
 $Comp
-L COM-09032:COM-09032 U1
+L Joystick_Follower_Hat-rescue:COM-09032-COM-09032 U1
 U 1 1 5F790376
 P 7725 3800
