File: Hardware/Joystick_Follower_Hat/Joystick_Follower_Hat.kicad_pcb (KiCad board)
At the start: 2 copper layers, 21 parts, among them SW1 SW_Push, SW2 SW_Push, SW3 SW_Push, SW4 SW_Push, U1 COM-09032

Commit message: PCB name change
Other:
- board text added: "Joystick Follower REV A SDSU Mechatronics"
- board text removed: "Joystick Follower REV A SDSU Mechatronics Designed By: Tristan Richmond & David Walker-Howell"

Commit message: sUpdated Gerbers
Routing:
- net Net-(A1-Pad19): track 74.8 -> 73.2 mm
